Commit message: make the ramp and door obstacle dependant on a ramp_up_slope and ramp_down_slope parameter

File: ros1/src/march_simulation/obstacles/ramp_and_door.xacro (robot description, xacro)
@@ -8,7 +8,9 @@
     <xacro:property name="platform_length" default="2.920"/>
     <xacro:property name="platform_width" default="1.4"/>
-    <xacro:property name="ramp_up_length" default="1.403"/>
-    <xacro:property name="ramp_down_length" default="1.854"/>
+    <xacro:property name="ramp_up_length" default="3.0"/>
     <xacro:property name="distance_to_origin" default="0.4"/>
+    <xacro:property name="ramp_up_slope" default="${radians(20)}"/>
+    <xacro:property name="ramp_down_slope" value="${radians(20)}"/>
+    <xacro:property name="ramp_down_length" default="${sin(ramp_up_slope) * ramp_up_length / sin(ramp_down_slope)}"/>
     <xacro:property name="parent_name" value="world"/>
     <xacro:property name="mu1" value="1.0"/>
@@ -86,18 +88,23 @@
     </gazebo>
     <!-- Joints -->
-    <joint name="joint_0" type="fixed">
+    <joint name="joint_0" type="fixed"> <!-- Ensure the ramp up side just above ground, and 0.4 m away from origin -->
         <parent link="${parent_name}"/>
+        <child link="ramp_up"/>
+        <origin xyz="${-1 * cos(radians(45) - ramp_up_slope) * ramp_up_length / sqrt(2) - distance_to_origin} 0
+                     ${-1 * sin(radians(45) - ramp_up_slope) * ramp_up_length / sqrt(2)}" rpy="0 ${ramp_up_slope} 0"/>
+    </joint>
+    <joint name="joint_1" type="fixed"> <!-- Let platform be straight, and smoothly connect it to the ramp up -->
+        <parent link="ramp_up"/>
         <child link="platform"/>
-        <origin xyz="-3.2 0 ${platform_height / 2}" rpy="0 0 0"/>
-    </joint>
-    <joint name="joint_1" type="fixed">
-        <parent link="platform"/>
-        <child link="ramp_up"/>
-        <origin xyz="1.875 0 -0.659" rpy="0 0.35 0"/>
+        <origin xyz="${-1 * ramp_up_length / 2 - cos(ramp_up_slope) * platform_length / 2 + sin(ramp_up_slope) * platform_height / 2} 0
+        ${ramp_up_length / 2 - sin(ramp_up_slope) * platform_length / 2 - cos(ramp_up_slope) * platform_height / 2}" rpy="0 ${-1 * ramp_up_slope} 0"/>
     </joint>
     <joint name="joint_2" type="fixed">
         <parent link="platform"/>
         <child link="ramp_down"/>
-        <origin xyz="-2.115 0 -0.895" rpy="0 -0.26 0"/>
+        <origin xyz="${-1 * platform_length / 2 - cos(radians(45) + ramp_down_slope) * ramp_down_length / sqrt(2)} 0
+        ${platform_height / 2 - sin(radians(45) + ramp_down_slope) * ramp_down_length / sqrt(2)}" rpy="0 ${-1 * ramp_down_slope} 0"/>
     </joint>
 </robot>
+<!--         <origin xyz="${-1 * sin(radians(45) - ramp_up_slope) * (ramp_up_length / sqrt(2)) - platform_length / 2} 0
+        ${cos(radians(45) - ramp_up_slope) * (ramp_up_length / sqrt(2)) - platform_height / 2}" rpy="0 ${-1 * ramp_up_slope} 0"/> -->
