Commit message: move CoM forward better

File: ros1/src/simulation/march_simulation/obstacles/ramp_and_door.xacro (robot description, xacro)
@@ -10,6 +10,6 @@
     <xacro:property name="ramp_up_length" default="3.0"/>
     <xacro:property name="distance_to_origin" default="0.4"/>
-    <xacro:property name="ramp_up_slope" default="${radians(20)}"/>
-    <xacro:property name="ramp_down_slope" value="${radians(20)}"/>
+    <xacro:property name="ramp_up_slope" default="${radians(15)}"/>
+    <xacro:property name="ramp_down_slope" value="${radians(15)}"/>
     <xacro:property name="ramp_down_length" default="${sin(ramp_up_slope) * ramp_up_length / sin(ramp_down_slope)}"/>
     <xacro:property name="parent_name" value="world"/>
