Commit message: finish collision and visual

File: ros1/src/march_description/urdf/march4_chain.xacro (robot description, xacro)
@@ -277,4 +277,5 @@
         </collision>
     </link>
+   <!-- Left Moving Hip-->
     <link name="hip_aa_frame_left_front">
         <inertial>
@@ -293,4 +294,178 @@
             <geometry>
                 <box size="${hip_aa_frame_width} ${width} ${width}"/>
+            </geometry>
+        </collision>
+    </link>
+    <link name="hip_aa_frame_left_side">
+        <visual>
+            <origin xyz="${-hip_aa_frame_width} ${hip_aa_frame_height+hip_base_height/2} 0" rpy="0 0 ${pi}"/>
+            <geometry>
+                <mesh filename="package://march_description/urdf/stl-files/LeftHAA.stl" scale="1 1 1"/>
+            </geometry>
+            <material name="blue"/>
+        </visual>
+        <collision>
+            <origin xyz="0 ${hip_aa_frame_height/2} 0" rpy="0 0 0"/>
+            <geometry>
+                <box size="${width} ${hip_aa_frame_height} ${width}"/>
+            </geometry>
+        </collision>
+    </link>
+    <!-- hip !-->
+    <link name="hip_base">
+        <visual>
+            <origin xyz="0 ${hip_base_height/2} 0" rpy="0 0 ${pi}"/>
+            <geometry>
+                <mesh filename="package://march_description/urdf/stl-files/HipBase.stl" scale="1 1 1"/>
+            </geometry>
+            <material name="blue"/>
+        </visual>
+        <inertial>
+            <origin xyz="${hip_base_com_x} ${hip_base_com_y} ${hip_base_com_z}" rpy="0 0 0"/>
+            <mass value="${hip_base_mass}"/>
+            <inertia
+                    ixx="${hip_base_Ixx}"
+                    ixy="${hip_base_Ixy}"
+                    ixz="${hip_base_Ixz}"
+                    iyy="${hip_base_Iyy}"
+                    iyz="${hip_base_Iyz}"
+                    izz="${hip_base_Izz}" />
+        </inertial>
+        <collision>
+            <origin xyz="0 ${hip_base_height/2} 0" rpy="0 0 0"/>
+            <geometry>
+                <box size="${width} ${hip_base_height} ${width}"/>
+            </geometry>
+        </collision>
+    </link>
+    <link name="hip_aa_frame_right_side">
+        <visual>
+            <origin xyz="${-hip_aa_frame_width} ${-hip_base_height/2} 0" rpy="0 0 ${pi}"/>
+            <geometry>
+                <mesh filename="package://march_description/urdf/stl-files/RightHAA.stl" scale="1 1 1"/>
+            </geometry>
+            <material name="blue"/>
+        </visual>
+        <collision>
+            <origin xyz="0 ${hip_aa_frame_height/2} 0" rpy="0 0 0"/>
+            <geometry>
+                <box size="${width} ${hip_aa_frame_height} ${width}"/>
+            </geometry>
+        </collision>
+    </link>
+	<link name="hip_aa_frame_right_front">
+        <inertial>
+            <origin xyz="${hip_aa_com_x} ${hip_aa_com_y} ${hip_aa_com_z}" rpy="0 0 0"/>
+            <mass value="${hip_aa_mass}"/>
+            <inertia
+                    ixx="${hip_aa_Ixx}"
+                    ixy="${hip_aa_Ixy}"
+                    ixz="${hip_aa_Ixz}"
+                    iyy="${hip_aa_Iyy}"
+                    iyz="${hip_aa_Iyz}"
+                    izz="${hip_aa_Izz}" />
+        </inertial>
+        <collision>
+            <origin xyz="${-hip_aa_frame_width/2} 0 0" rpy="0 0 0"/>
+            <geometry>
+                <box size="${hip_aa_frame_width} ${width} ${width}"/>
+            </geometry>
+        </collision>
+    </link>
+        <!-- Upper Leg Right-->
+    <link name="upper_leg_right">
+        <visual>
+            <origin xyz="0 ${-hip_base_height/2 - hip_aa_frame_height + upper_leg_offset} 0" rpy="0 0 ${pi}"/>
+            <geometry>
+                <mesh filename="package://march_description/urdf/stl-files/UpperRightLeg.stl" scale="1 1 1"/>
+            </geometry>
+            <material name="blue"/>
+        </visual>
+        <inertial>
+            <origin xyz="${upper_leg_com_x} ${upper_leg_com_y} ${upper_leg_com_z}" rpy="0 0 0"/>
+            <mass value="${upper_leg_mass}"/>
+            <inertia
+                    ixx="${upper_leg_Ixx}"
+                    ixy="${upper_leg_Ixy}"
+                    ixz="${upper_leg_Ixz}"
+                    iyy="${upper_leg_Iyy}"
+                    iyz="${upper_leg_Iyz}"
+                    izz="${upper_leg_Izz}" />
+        </inertial>
+        <collision>
+            <origin xyz="0 0 ${-upper_leg_height/2}" rpy="0 0 0"/>
+            <geometry>
+                <box size="${width} ${width} ${upper_leg_height}"/>
+            </geometry>
+        </collision>
+    </link>
+    <!-- Lower Leg Right -->
+    <link name="lower_leg_right">
+        <visual>
+            <origin
+                xyz="0 ${-hip_base_height/2 - hip_aa_frame_height + upper_leg_offset} ${upper_leg_height}"
+                rpy="0 0 ${pi}"
+            />
+            <geometry>
+                <mesh filename="package://march_description/urdf/stl-files/LowerRightLeg.stl" scale="1 1 1"/>
+            </geometry>
+            <material name="blue"/>
+        </visual>
+        <inertial>
+            <origin xyz="${lower_leg_com_x} ${lower_leg_com_y} ${lower_leg_com_z}" rpy="0 0 0"/>
+            <mass value="${lower_leg_mass}"/>
+            <inertia
+                    ixx="${lower_leg_Ixx}"
+                    ixy="${lower_leg_Ixy}"
+                    ixz="${lower_leg_Ixz}"
+                    iyy="${lower_leg_Iyy}"
+                    iyz="${lower_leg_Iyz}"
+                    izz="${lower_leg_Izz}" />
+        </inertial>
+        <collision>
+            <origin xyz="0 0 ${-lower_leg_height/2}" rpy="0 0 0"/>
+            <geometry>
+                <box size="${width} ${width} ${lower_leg_height}"/>
+            </geometry>
+        </collision>
+    </link>
+    <!-- Ankle Plate Right -->
+    <link name="ankle_plate_right">
+        <visual>
+            <origin
+                xyz="0
+                    ${-hip_base_height/2 - hip_aa_frame_height+ upper_leg_offset + ankle_plate_offset}
+                    ${foot_scale * (upper_leg_height + lower_leg_height)}"
+                rpy="0 0 ${pi}"/>
+            />
+            <geometry>
+                <mesh filename="package://march_description/urdf/stl-files/RightFoot.stl" scale="1 1 ${foot_scale}"/>
+            </geometry>
+            <material name="blue"/>
+        </visual>
+        <collision>
+            <origin xyz="0 0 ${-ankle_plate_height/2}" rpy="0 0 0"/>
+            <geometry>
+                <box size="${width} ${width} ${ankle_plate_height}"/>
+            </geometry>
+        </collision>
+    </link>
+    <!-- Foot Right -->
+    <link name="foot_right">
+        <inertial>
+            <origin xyz="${foot_com_x} ${foot_com_y} ${foot_com_z}" rpy="0 0 0"/>
+            <mass value="${foot_mass}"/>
+            <inertia
+                    ixx="${foot_Ixx}"
+                    ixy="${foot_Ixy}"
+                    ixz="${foot_Ixz}"
+                    iyy="${foot_Iyy}"
+                    iyz="${foot_Iyz}"
+                    izz="${foot_Izz}" />
+        </inertial>
+        <collision>
+            <origin xyz="${(-foot_height_forward+foot_height_backward)/2} 0 0" rpy="0 0 0"/>
+            <geometry>
+                <box size="${foot_height_forward+foot_height_backward} ${width} ${width}"/>
             </geometry>
         </collision>
@@ -337,5 +512,5 @@
         <parent link="upper_leg_left"/>
         <child link="hip_aa_frame_left_front"/>
-        <origin xyz="0 0 ${upper_leg_height}" rpy="0 0 0"/>
+        <origin xyz="0 ${-upper_leg_offset} ${upper_leg_height}" rpy="0 0 0"/>
         <axis xyz="0 1 0"/>
         <limit velocity="${hip_fe_velocity_limit}"
@@ -348,4 +523,89 @@
                            k_velocity="${k_velocity_value_hfe}" />
     </joint>
+    <joint name="left_hip_angle" type="fixed">
+        <parent link="hip_aa_frame_left_front"/>
+        <child link="hip_aa_frame_left_side"/>
+        <origin xyz="${hip_aa_frame_width} 0 0" rpy="0 0 0"/>
+    </joint>
+    <joint name="left_hip_aa" type="revolute">
+        <parent link="hip_aa_frame_left_side"/>
+        <child link="hip_base"/>
+        <origin xyz="0 ${hip_aa_frame_height} 0" rpy="0 0 0"/>
+        <axis xyz="-1 0 0"/>
+        <limit velocity="${hip_aa_velocity_limit}"
+               effort="${hip_aa_effort_limit}"
+               lower="${left_hip_aa_rotation_lower_limit}"
+               upper="${left_hip_aa_rotation_upper_limit}"/>
+        <safety_controller soft_lower_limit="${left_hip_aa_rotation_lower_limit + hip_aa_soft_buffer}"
+                           soft_upper_limit="${left_hip_aa_rotation_upper_limit - hip_aa_soft_buffer}"
+                           k_position="${k_position_value_haa}"
+                           k_velocity="${k_velocity_value_haa}" />
+    </joint>
+    <joint name="right_hip_aa" type="revolute">
+        <parent link="hip_base"/>
+        <child link="hip_aa_frame_right_side"/>
+        <origin xyz="0 ${hip_base_height} 0" rpy="0 0 0"/>
+        <axis xyz="1 0 0"/>
+        <limit velocity="${hip_aa_velocity_limit}"
+               effort="${hip_aa_effort_limit}"
+               lower="${right_hip_aa_rotation_lower_limit}"
+               upper="${right_hip_aa_rotation_upper_limit}"/>
+        <safety_controller soft_lower_limit="${right_hip_aa_rotation_lower_limit + hip_aa_soft_buffer}"
+                           soft_upper_limit="${right_hip_aa_rotation_upper_limit - hip_aa_soft_buffer}"
+                           k_position="${k_position_value_haa}"
+                           k_velocity="${k_velocity_value_haa}" />
+    </joint>
+    <joint name="right_hip_angle" type="fixed">
+        <parent link="hip_aa_frame_right_side"/>
+        <child link="hip_aa_frame_right_front"/>
+        <origin xyz="0 ${hip_aa_frame_height} 0" rpy="0 0 0"/>
+    </joint>
+    <joint name="right_hip_fe" type="revolute">
+        <parent link="hip_aa_frame_right_front"/>
+        <child link="upper_leg_right"/>
+        <origin xyz="${-hip_aa_frame_width} ${-upper_leg_offset} 0" rpy="0 0 0"/>
+        <axis xyz="0 1 0"/>
+        <limit velocity="${hip_fe_velocity_limit}"
+               effort="${hip_fe_effort_limit}"
+               lower="${right_hip_fe_rotation_lower_limit}"
+               upper="${right_hip_fe_rotation_upper_limit}"/>
+        <safety_controller soft_lower_limit="${right_hip_fe_rotation_lower_limit + hip_fe_soft_buffer}"
+                           soft_upper_limit="${right_hip_fe_rotation_upper_limit - hip_fe_soft_buffer}"
+                           k_position="${k_position_value_hfe}"
+                           k_velocity="${k_velocity_value_hfe}" />
+    </joint>
+    <joint name="right_knee" type="revolute">
+        <parent link="upper_leg_right"/>
+        <child link="lower_leg_right"/>
+        <origin xyz="0 0 ${-upper_leg_height}" rpy="0 0 0"/>
+        <axis xyz="0 -1 0"/>
+        <limit velocity="${knee_velocity_limit}"
+               effort="${knee_effort_limit}"
+               lower="${right_knee_rotation_lower_limit}"
+               upper="${right_knee_rotation_upper_limit}"/>
+        <safety_controller soft_lower_limit="${right_knee_rotation_lower_limit + knee_extension_soft_buffer}"
+                           soft_upper_limit="${right_knee_rotation_upper_limit - knee_flexion_soft_buffer}"
+                           k_position="${k_position_value_kfe}"
+                           k_velocity="${k_velocity_value_kfe}" />
+    </joint>
+    <joint name="right_ankle" type="revolute">
+        <parent link="lower_leg_right"/>
+        <child link="ankle_plate_right"/>
+        <origin xyz="0 ${-ankle_plate_offset} ${-lower_leg_height}" rpy="0 0 0"/>
+        <axis xyz="0 1 0"/>
+        <limit velocity="${ankle_velocity_limit}"
+               effort="${ankle_effort_limit}"
+               lower="${right_ankle_rotation_lower_limit}"
+               upper="${right_ankle_rotation_upper_limit}"/>
+        <safety_controller soft_lower_limit="${right_ankle_rotation_lower_limit + ankle_plantarflexion_soft_buffer}"
+                           soft_upper_limit="${right_ankle_rotation_upper_limit - ankle_dorsalflexion_soft_buffer}"
+                           k_position="${k_position_value_adpf}"
+                           k_velocity="${k_velocity_value_adpf}" />
+    </joint>
+    <joint name="right_foot_angle" type="fixed">
+        <parent link="ankle_plate_right"/>
+        <child link="foot_right"/>
+        <origin xyz="0 0 ${-ankle_plate_height}" rpy="0 0 0"/>
+    </joint>
     <!-- ROS Control plugin for Gazebo -->
     <transmission name="left_hip_aa">

Commit message: Fix gazebo robot model by adding inertia

File: ros1/src/march_description/urdf/march4_chain.xacro (robot description, xacro)
@@ -199,5 +199,4 @@
         <fdir1>1 0 0</fdir1>
     </gazebo>
-    <!-- Ankle plate Left -->
     <link name="ankle_plate_left">
         <visual>
@@ -205,5 +204,5 @@
                 xyz="0
                      ${hip_base_height/2 + hip_aa_frame_height - upper_leg_offset - ankle_plate_offset}
-                     ${foot_scale * (upper_leg_height + lower_leg_height + ankle_plate_height)}"
+                     ${foot_scale * (upper_leg_height + lower_leg_height + ankle_plate_height) - foot_height_backward}"
                 rpy="0 0 ${pi}"
             />
@@ -219,6 +218,17 @@
             </geometry>
         </collision>
-    </link>
-    <!-- Lower Leg Left -->
+        <inertial>
+            <origin xyz="0 0 0" rpy="0 0 0"/>
+            <mass value="1"/> <!-- ARBITRARY NON-ZERO VALUE-->
+            <inertia
+                    ixx="${lower_leg_Ixx}"
+                    ixy="${-lower_leg_Ixy}"
+                    ixz="${lower_leg_Ixz}"
+                    iyy="${lower_leg_Iyy}"
+                    iyz="${-lower_leg_Iyz}"
+                    izz="${lower_leg_Izz}"
+                />
+        </inertial>
+    </link>
     <link name="lower_leg_left">
         <visual>
@@ -250,5 +260,4 @@
         </collision>
     </link>
-    <!-- Upper Leg Left-->
     <link name="upper_leg_left">
         <visual>
@@ -277,5 +286,4 @@
         </collision>
     </link>
-   <!-- Left Moving Hip-->
     <link name="hip_aa_frame_left_front">
         <inertial>
@@ -311,6 +319,17 @@
             </geometry>
         </collision>
-    </link>
-    <!-- hip !-->
+        <inertial>
+            <origin xyz="0 0 0" rpy="0 0 0"/>
+            <mass value="1"/> <!-- ARBITRARY NON-ZERO VALUE-->
+            <inertia
+                    ixx="${lower_leg_Ixx}"
+                    ixy="${-lower_leg_Ixy}"
+                    ixz="${lower_leg_Ixz}"
+                    iyy="${lower_leg_Iyy}"
+                    iyz="${-lower_leg_Iyz}"
+                    izz="${lower_leg_Izz}"
+                />
+        </inertial>
+    </link>
     <link name="hip_base">
         <visual>
@@ -373,5 +392,4 @@
         </collision>
     </link>
-        <!-- Upper Leg Right-->
     <link name="upper_leg_right">
         <visual>
@@ -400,5 +418,4 @@
         </collision>
     </link>
-    <!-- Lower Leg Right -->
     <link name="lower_leg_right">
         <visual>
@@ -430,5 +447,4 @@
         </collision>
     </link>
-    <!-- Ankle Plate Right -->
     <link name="ankle_plate_right">
         <visual>
@@ -451,5 +467,4 @@
         </collision>
     </link>
-    <!-- Foot Right -->
     <link name="foot_right">
         <inertial>
@@ -485,5 +500,5 @@
         <child link="lower_leg_left"/>
         <origin xyz="0 ${-ankle_plate_offset} ${ankle_plate_height}" rpy="0 0 0"/>
-        <axis xyz="0 1 0"/>
+        <axis xyz="0 -1 0"/>
         <limit velocity="${ankle_velocity_limit}"
                effort="${ankle_effort_limit}"
@@ -499,5 +514,5 @@
         <child link="upper_leg_left"/>
         <origin xyz="0 0 ${lower_leg_height}" rpy="0 0 0"/>
-        <axis xyz="0 -1 0"/>
+        <axis xyz="0 1 0"/>
         <limit velocity="${knee_velocity_limit}"
                effort="${knee_effort_limit}"
@@ -513,5 +528,5 @@
         <child link="hip_aa_frame_left_front"/>
         <origin xyz="0 ${-upper_leg_offset} ${upper_leg_height}" rpy="0 0 0"/>
-        <axis xyz="0 1 0"/>
+        <axis xyz="0 -1 0"/>
         <limit velocity="${hip_fe_velocity_limit}"
                effort="${hip_fe_effort_limit}"
@@ -532,5 +547,5 @@
         <child link="hip_base"/>
         <origin xyz="0 ${hip_aa_frame_height} 0" rpy="0 0 0"/>
-        <axis xyz="-1 0 0"/>
+        <axis xyz="1 0 0"/>
         <limit velocity="${hip_aa_velocity_limit}"
                effort="${hip_aa_effort_limit}"
@@ -609,4 +624,31 @@
     </joint>
     <!-- ROS Control plugin for Gazebo -->
+    <transmission name="left_ankle">
+        <type>transmission_interface/SimpleTransmission</type>
+        <joint name="left_ankle">
+            <hardwareInterface>hardware_interface/EffortJointInterface</hardwareInterface>
+        </joint>
+        <actuator name="left_ankle_motor">
+            <mechanicalReduction>200</mechanicalReduction>
+        </actuator>
+    </transmission>
+    <transmission name="left_knee">
+        <type>transmission_interface/SimpleTransmission</type>
+        <joint name="left_knee">
+            <hardwareInterface>hardware_interface/EffortJointInterface</hardwareInterface>
+        </joint>
+        <actuator name="left_knee_motor">
+            <mechanicalReduction>101</mechanicalReduction>
+        </actuator>
+    </transmission>
+    <transmission name="left_hip_fe">
+        <type>transmission_interface/SimpleTransmission</type>
+        <joint name="left_hip_fe">
+            <hardwareInterface>hardware_interface/EffortJointInterface</hardwareInterface>
+        </joint>
+        <actuator name="left_hip_fe_motor">
+            <mechanicalReduction>101</mechanicalReduction>
+        </actuator>
+    </transmission>
     <transmission name="left_hip_aa">
         <type>transmission_interface/SimpleTransmission</type>
@@ -618,31 +660,4 @@
         </actuator>
     </transmission>
-    <transmission name="left_hip_fe">
-        <type>transmission_interface/SimpleTransmission</type>
-        <joint name="left_hip_fe">
-            <hardwareInterface>hardware_interface/EffortJointInterface</hardwareInterface>
-        </joint>
-        <actuator name="left_hip_fe_motor">
-            <mechanicalReduction>101</mechanicalReduction>
-        </actuator>
-    </transmission>
-    <transmission name="left_knee">
-        <type>transmission_interface/SimpleTransmission</type>
-        <joint name="left_knee">
-            <hardwareInterface>hardware_interface/EffortJointInterface</hardwareInterface>
-        </joint>
-        <actuator name="left_knee_motor">
-            <mechanicalReduction>101</mechanicalReduction>
-        </actuator>
-    </transmission>
-    <transmission name="left_ankle">
-        <type>transmission_interface/SimpleTransmission</type>
-        <joint name="left_ankle">
-            <hardwareInterface>hardware_interface/EffortJointInterface</hardwareInterface>
-        </joint>
-        <actuator name="left_ankle_motor">
-            <mechanicalReduction>200</mechanicalReduction>
-        </actuator>
-    </transmission>
     <transmission name="right_hip_aa">
         <type>transmission_interface/SimpleTransmission</type>

Commit message: Correct CoM of all links with respect to new origin

File: ros1/src/march_description/urdf/march4_chain.xacro (robot description, xacro)
@@ -76,5 +76,5 @@
          the y coordinate will be inverted for the left leg. -->
     <xacro:property name="hip_base_com_x" value="${-hip_aa_frame_width + 0.147989}"/>
-    <xacro:property name="hip_base_com_y" value="0.016341"/>
+    <xacro:property name="hip_base_com_y" value="${hip_base_height/2 + 0.016341}"/>
     <xacro:property name="hip_base_com_z" value="0.147761"/>
     <xacro:property name="hip_aa_com_x" value="${-hip_aa_frame_width + 0.108094}"/>
@@ -176,5 +176,5 @@
     <link name="foot_left">
         <inertial>
-            <origin xyz="${foot_com_x} ${-foot_com_y} ${foot_com_z}" rpy="0 0 0"/>
+            <origin xyz="${foot_com_x} ${-foot_com_y} ${foot_com_z + ankle_plate_height/2}" rpy="0 0 0"/>
             <mass value="${foot_mass}"/>
             <inertia
@@ -243,5 +243,5 @@
         </visual>
         <inertial>
-            <origin xyz="${lower_leg_com_x} ${-lower_leg_com_y} ${lower_leg_com_z}" rpy="0 0 0"/>
+            <origin xyz="${lower_leg_com_x} ${-lower_leg_com_y} ${lower_leg_com_z + lower_leg_height}" rpy="0 0 0"/>
             <mass value="${lower_leg_mass}"/>
             <inertia
@@ -269,5 +269,5 @@
         </visual>
         <inertial>
-            <origin xyz="${upper_leg_com_x} ${-upper_leg_com_y} ${upper_leg_com_z}" rpy="0 0 0"/>
+            <origin xyz="${upper_leg_com_x} ${-upper_leg_com_y} ${upper_leg_com_z + upper_leg_height}" rpy="0 0 0"/>
             <mass value="${upper_leg_mass}"/>
             <inertia
@@ -288,5 +288,5 @@
     <link name="hip_aa_frame_left_front">
         <inertial>
-            <origin xyz="${hip_aa_com_x} ${-hip_aa_com_y} ${hip_aa_com_z}" rpy="0 0 0"/>
+            <origin xyz="${hip_aa_com_x + hip_aa_frame_width} ${-hip_aa_com_y} ${hip_aa_com_z}" rpy="0 0 0"/>
             <mass value="${hip_aa_mass}"/>
             <inertia
@@ -490,4 +490,5 @@
         <parent link="${parent_name}"/>
         <child link="foot_left"/>
+        <origin xyz="0 0 ${width/2}" rpy="0 0 0"/>
     </joint>
     <joint name="left_foot_angle" type="fixed">
