Commit message: Copy MarchV changesn

File: ros1/src/march_description/urdf/test_joint_rotational.xacro (robot description, xacro)
@@ -11,5 +11,5 @@
     <xacro:property name="joint_lower_limit" value="-0.5363"/> <!-- rad -->
     <xacro:property name="joint_upper_limit" value="0.5363"/> <!-- rad -->
-    <xacro:property name="joint_effort_limit" value="21840"/> <!-- IU = 20 A -->
+    <xacro:property name="joint_effort_limit" value="28"/> <!-- IU = 20 A -->
     <xacro:property name="joint_velocity_limit" value="2.0"/> <!-- rad/s -->
     <xacro:property name="hover_height" value="0.5"/>
@@ -29,5 +29,5 @@
         <axis xyz="0 1 0"/>
         <limit velocity="${joint_velocity_limit}" effort="${joint_effort_limit}" lower="${joint_lower_limit}" upper="${joint_upper_limit}"/>
-        <safety_controller soft_lower_limit="${joint_lower_limit + joint_buffer}" soft_upper_limit="${joint_upper_limit - joint_buffer}" k_position="5" k_velocity="20000" />
+        <safety_controller soft_lower_limit="${joint_lower_limit + joint_buffer}" soft_upper_limit="${joint_upper_limit - joint_buffer}" k_position="5" k_velocity="24.4" />
     </joint>
     <!-- give colors to some links in gazebo -->

Commit message: Change order of setting control mode

File: ros1/src/march_description/urdf/test_joint_rotational.xacro (robot description, xacro)
@@ -12,5 +12,5 @@
     <xacro:property name="joint_upper_limit" value="0.5363"/> <!-- rad -->
     <xacro:property name="joint_effort_limit" value="28"/> <!-- IU = 20 A -->
-    <xacro:property name="joint_velocity_limit" value="2.0"/> <!-- rad/s -->
+    <xacro:property name="joint_velocity_limit" value="10.0"/> <!-- rad/s -->
     <xacro:property name="hover_height" value="0.5"/>
     <!-- Import all Gazebo-customization elements, including Gazebo colors -->

Commit message: Add final changes

File: ros1/src/march_description/urdf/test_joint_rotational.xacro (robot description, xacro)
@@ -9,6 +9,6 @@
     <xacro:property name="bar_width" value="0.05"/>
     <xacro:property name="joint_buffer" value="${3*pi/180}"/> <!-- rad -->
-    <xacro:property name="joint_lower_limit" value="-0.5363"/> <!-- rad -->
-    <xacro:property name="joint_upper_limit" value="0.5363"/> <!-- rad -->
+    <xacro:property name="joint_lower_limit" value="-1"/> <!-- rad -->
+    <xacro:property name="joint_upper_limit" value="1"/> <!-- rad -->
     <xacro:property name="joint_effort_limit" value="28"/> <!-- IU = 20 A -->
     <xacro:property name="joint_velocity_limit" value="10.0"/> <!-- rad/s -->
