Commit message: Allow rviz and gazebo to be run from same urdf file by altering mesh_basepath conditionally

File: ros2/src/shared/march_description/urdf/march4_position.xacro (robot description, xacro)
@@ -2,7 +2,4 @@
 <!-- Revolute-Revolute Manipulator -->
 <robot name="march" xmlns:xacro="http://www.ros.org/wiki/xacro">
-    <!-- An argument that makes sure the march.gazebo is loaded only when launching the simulation and not during build,
-            because during build the march_description package can not be found-->
-    <xacro:arg name="build" default="false"/>
     <!-- Switch between airgaiting or standing on the ground-->
     <!-- Value set to: 'world' fixes the robot to the world-->
@@ -10,4 +7,13 @@
     the hover_height to 0.0. Set ground_gait to true to ground gait in simulation.-->
     <xacro:arg name="ground_gait" default="false"/>
+    <!-- The meshes have to be loaded differently for rviz than for gazebo_ui-->
+    <!-- This argument is used to set the 'base_path' of the meshes-->
+    <xacro:arg name="gazebo_ui" default="true"/>
+    <xacro:if value="$(arg gazebo_ui)">
+        <xacro:property name="mesh_basepath" value="$(find march_description)"/>
+    </xacro:if>
+    <xacro:unless value="$(arg gazebo_ui)">
+        <xacro:property name="mesh_basepath" value="package://march_description"/>
+    </xacro:unless>
     <xacro:unless value="$(arg ground_gait)">
         <xacro:property name="parent_name" value="world"/>
@@ -169,13 +175,11 @@
     <!-- Import all Gazebo-customization elements, including Gazebo colors -->
     <!-- Import all Gazebo-customization elements, including Gazebo colors -->
-    <xacro:unless value="$(arg build)">
-        <gazebo>
-            <plugin name="gazebo_ros2_control" filename="libgazebo_ros2_control.so">
-                <robotNamespace>/march</robotNamespace>
-                <robotSimType>gazebo_ros2_control/DefaultRobotHWSim</robotSimType>
-                <parameters>$(find march_simulation)/config/position_control/march4.yaml</parameters>
-            </plugin>
-        </gazebo>
-    </xacro:unless>
+    <gazebo>
+        <plugin name="gazebo_ros2_control" filename="libgazebo_ros2_control.so">
+            <robotNamespace>/march</robotNamespace>
+            <robotSimType>gazebo_ros2_control/DefaultRobotHWSim</robotSimType>
+            <parameters>$(find march_simulation)/config/position_control/march4.yaml</parameters>
+        </plugin>
+    </gazebo>
     <material name="blue">
         <color rgba="0 0 0.6 1"/>
@@ -189,5 +193,5 @@
             <origin xyz="${-hip_aa_frame_width} 0 0" rpy="0 0 ${pi}"/>
             <geometry>
-                <mesh filename="package://march_description/urdf/stl-files/HipBase.stl" scale="1 1 1"/>
+                <mesh filename="${mesh_basepath}/urdf/stl-files/HipBase.stl" scale="1 1 1"/>
             </geometry>
             <material name="blue"/>
@@ -219,5 +223,5 @@
             <origin xyz="${-hip_aa_frame_width} ${hip_base_height/2} 0" rpy="0 0 ${pi}"/>
             <geometry>
-                <mesh filename="package://march_description/urdf/stl-files/LeftHAA.stl" scale="1 1 1"/>
+                <mesh filename="${mesh_basepath}/urdf/stl-files/LeftHAA.stl" scale="1 1 1"/>
             </geometry>
             <material name="blue"/>
@@ -254,5 +258,5 @@
             <origin xyz="0 ${hip_base_height/2 + hip_aa_frame_height - upper_leg_offset} 0" rpy="0 0 ${pi}"/>
             <geometry>
-                <mesh filename="package://march_description/urdf/stl-files/UpperLeftLeg.stl" scale="1 1 1"/>
+                <mesh filename="${mesh_basepath}/urdf/stl-files/UpperLeftLeg.stl" scale="1 1 1"/>
             </geometry>
             <material name="blue"/>
@@ -284,5 +288,5 @@
             />
             <geometry>
-                <mesh filename="package://march_description/urdf/stl-files/LowerLeftLeg.stl" scale="1 1 1"/>
+                <mesh filename="${mesh_basepath}/urdf/stl-files/LowerLeftLeg.stl" scale="1 1 1"/>
             </geometry>
             <material name="blue"/>
@@ -316,5 +320,5 @@
             />
             <geometry>
-                <mesh filename="package://march_description/urdf/stl-files/LeftFoot.stl" scale="1 1 ${foot_scale}"/>
+                <mesh filename="${mesh_basepath}/urdf/stl-files/LeftFoot.stl" scale="1 1 ${foot_scale}"/>
             </geometry>
             <material name="blue"/>
@@ -358,5 +362,5 @@
             <origin xyz="${-hip_aa_frame_width} ${-hip_base_height/2} 0" rpy="0 0 ${pi}"/>
             <geometry>
-                <mesh filename="package://march_description/urdf/stl-files/RightHAA.stl" scale="1 1 1"/>
+                <mesh filename="${mesh_basepath}/urdf/stl-files/RightHAA.stl" scale="1 1 1"/>
             </geometry>
             <material name="blue"/>
@@ -393,5 +397,5 @@
             <origin xyz="0 ${-hip_base_height/2 - hip_aa_frame_height + upper_leg_offset} 0" rpy="0 0 ${pi}"/>
             <geometry>
-                <mesh filename="package://march_description/urdf/stl-files/UpperRightLeg.stl" scale="1 1 1"/>
+                <mesh filename="${mesh_basepath}/urdf/stl-files/UpperRightLeg.stl" scale="1 1 1"/>
             </geometry>
             <material name="blue"/>
@@ -423,5 +427,5 @@
             />
             <geometry>
-                <mesh filename="package://march_description/urdf/stl-files/LowerRightLeg.stl" scale="1 1 1"/>
+                <mesh filename="${mesh_basepath}/urdf/stl-files/LowerRightLeg.stl" scale="1 1 1"/>
             </geometry>
             <material name="blue"/>
@@ -455,5 +459,5 @@
             />
             <geometry>
-                <mesh filename="package://march_description/urdf/stl-files/RightFoot.stl" scale="1 1 ${foot_scale}"/>
+                <mesh filename="${mesh_basepath}/urdf/stl-files/RightFoot.stl" scale="1 1 ${foot_scale}"/>
             </geometry>
             <material name="blue"/>
