Commit message: increase max effort and max velocity joints test

File: ros1/src/shared/march_description/urdf/march4.xacro (robot description, xacro)
@@ -20,5 +20,5 @@
     <!-- The max effort of the rotary joints is lower then the value corresponding to 25A, because short-circuit errors
     have occured while applying the theoretical max effort for a long time. -->
-    <xacro:arg name="max_effort_rotary" default="18000.0" />
+    <xacro:arg name="max_effort_rotary" default="28000.0" />
     <xacro:arg name="max_effort_linear" default="22932.0" />  <!-- = 28 A -->
     <xacro:property name="max_effort_rotary" value="$(arg max_effort_rotary)" />
@@ -138,5 +138,5 @@
     <xacro:property name="hip_fe_soft_buffer" value="${3*pi/180}"/> <!-- rad -->
     <xacro:property name="hip_fe_effort_limit" value="${max_effort_rotary}"/> <!-- IU -->
-    <xacro:property name="hip_fe_velocity_limit" value="2.0"/> <!-- rad/s -->
+    <xacro:property name="hip_fe_velocity_limit" value="3.6"/> <!-- rad/s -->
     <xacro:property name="left_hip_aa_rotation_lower_limit" value="${-18.54492188*pi/180}"/> <!-- rad -->
     <xacro:property name="left_hip_aa_rotation_upper_limit" value="${16.34765625*pi/180}"/> <!-- rad -->
@@ -145,5 +145,5 @@
     <xacro:property name="hip_aa_soft_buffer" value="${3.5*pi/180}"/> <!-- rad -->
     <xacro:property name="hip_aa_effort_limit" value="${max_effort_linear}"/> <!-- IU -->
-    <xacro:property name="hip_aa_velocity_limit" value="1.0"/> <!-- rad/s -->
+    <xacro:property name="hip_aa_velocity_limit" value="2"/> <!-- rad/s -->
     <xacro:property name="left_knee_rotation_lower_limit" value="${-5.012512207*pi/180}"/>
     <xacro:property name="left_knee_rotation_upper_limit" value="${112.4230957*pi/180}"/>
@@ -153,5 +153,5 @@
     <xacro:property name="knee_flexion_soft_buffer" value="${3*pi/180}"/> <!-- rad -->
     <xacro:property name="knee_effort_limit" value="${max_effort_rotary}"/> <!-- IU -->
-    <xacro:property name="knee_velocity_limit" value="2.5"/>
+    <xacro:property name="knee_velocity_limit" value="3.6"/>
     <xacro:property name="left_ankle_rotation_lower_limit" value="${-26.30401611*pi/180}"/>
     <xacro:property name="left_ankle_rotation_upper_limit" value="${15.88348389*pi/180}"/>
@@ -161,5 +161,5 @@
     <xacro:property name="ankle_plantarflexion_soft_buffer" value="${3*pi/180}"/> <!-- rad -->
     <xacro:property name="ankle_effort_limit" value="${max_effort_linear}"/> <!-- IU -->
-    <xacro:property name="ankle_velocity_limit" value="1.0"/>
+    <xacro:property name="ankle_velocity_limit" value="2"/>
     <xacro:property name="camera_link" value="0.05"/> <!-- Size of square 'camera' box -->
     <xacro:property name="axel_offset" value="0.05"/> <!-- Space btw top of beam and the each joint -->

Commit message: increase max vel rotational joints :

File: ros1/src/shared/march_description/urdf/march4.xacro (robot description, xacro)
@@ -138,5 +138,5 @@
     <xacro:property name="hip_fe_soft_buffer" value="${3*pi/180}"/> <!-- rad -->
     <xacro:property name="hip_fe_effort_limit" value="${max_effort_rotary}"/> <!-- IU -->
-    <xacro:property name="hip_fe_velocity_limit" value="3.6"/> <!-- rad/s -->
+    <xacro:property name="hip_fe_velocity_limit" value="5"/> <!-- rad/s -->
     <xacro:property name="left_hip_aa_rotation_lower_limit" value="${-18.54492188*pi/180}"/> <!-- rad -->
     <xacro:property name="left_hip_aa_rotation_upper_limit" value="${16.34765625*pi/180}"/> <!-- rad -->
@@ -145,5 +145,5 @@
     <xacro:property name="hip_aa_soft_buffer" value="${3.5*pi/180}"/> <!-- rad -->
     <xacro:property name="hip_aa_effort_limit" value="${max_effort_linear}"/> <!-- IU -->
-    <xacro:property name="hip_aa_velocity_limit" value="2"/> <!-- rad/s -->
+    <xacro:property name="hip_aa_velocity_limit" value="3"/> <!-- rad/s -->
     <xacro:property name="left_knee_rotation_lower_limit" value="${-5.012512207*pi/180}"/>
     <xacro:property name="left_knee_rotation_upper_limit" value="${112.4230957*pi/180}"/>
@@ -153,5 +153,5 @@
     <xacro:property name="knee_flexion_soft_buffer" value="${3*pi/180}"/> <!-- rad -->
     <xacro:property name="knee_effort_limit" value="${max_effort_rotary}"/> <!-- IU -->
-    <xacro:property name="knee_velocity_limit" value="3.6"/>
+    <xacro:property name="knee_velocity_limit" value="5"/>
     <xacro:property name="left_ankle_rotation_lower_limit" value="${-26.30401611*pi/180}"/>
     <xacro:property name="left_ankle_rotation_upper_limit" value="${15.88348389*pi/180}"/>

Commit message: Re-add camera to xacro

File: ros1/src/shared/march_description/urdf/march4.xacro (robot description, xacro)
@@ -662,4 +662,8 @@
         <origin xyz="0 0 ${-ankle_plate_height}" rpy="0 0 0"/>
     </joint>
+    <xacro:include filename="$(find realsense2_description)/urdf/_d435.urdf.xacro" />
+    <xacro:sensor_d435 parent="upper_leg_left">
+        <origin xyz="0 0 0" rpy="0 0 3.1416"/>
+    </xacro:sensor_d435>
     <!-- ROS Control plugin for Gazebo -->
     <transmission name="left_hip_aa">

Commit message: Working node, except for error caused by pcl conversions

File: ros1/src/shared/march_description/urdf/march4.xacro (robot description, xacro)
@@ -7,4 +7,5 @@
     the hover_height to 0.0. Set ground_gait to true to ground gait in simulation.-->
     <xacro:arg name="ground_gait" default="false"/>
+    <xacro:arg name="realsense" default="false"/>
     <xacro:unless value="$(arg ground_gait)">
         <xacro:property name="parent_name" value="world"/>
@@ -662,8 +663,10 @@
         <origin xyz="0 0 ${-ankle_plate_height}" rpy="0 0 0"/>
     </joint>
-    <xacro:include filename="$(find realsense2_description)/urdf/_d435.urdf.xacro" />
-    <xacro:sensor_d435 parent="upper_leg_left">
-        <origin xyz="0 0 0" rpy="0 0 3.1416"/>
-    </xacro:sensor_d435>
+    <xacro:if value="$(arg realsense)">
+        <xacro:include filename="$(find realsense2_description)/urdf/_d435.urdf.xacro" />
+        <xacro:sensor_d435 parent="upper_leg_left">
+            <origin xyz="0 0 0" rpy="0 0 3.1416"/>
+        </xacro:sensor_d435>
+    </xacro:if>
     <!-- ROS Control plugin for Gazebo -->
     <transmission name="left_hip_aa">
