Commit message: Make hipbase fixed to world

File: ros1/src/shared/march_description/urdf/march4_chain.xacro (robot description, xacro)
@@ -174,4 +174,5 @@
     <!-- New order of links; The new robot model is a chain, with the origin in the 'Foot left' !-->
     <!-- Foot Left -->
+    <link name="dummy_link"/>
     <link name="foot_left">
         <inertial>
@@ -487,8 +488,15 @@
     </link>
     <!-- Joints -->
+    <!--
     <joint name = "foot_to_world" type="fixed">
         <parent link="${parent_name}"/>
         <child link="foot_left"/>
         <origin xyz="0 0 ${width/2}" rpy="0 0 0"/>
+    </joint>-->
+    <!-- This dummy joint is a workaround, since KDL does not support root links (foot_left) with inertias-->
+    <joint name="dummy_joint" type="fixed">
+        <parent link="dummy_link"/>
+        <child link="foot_left"/>
+        <origin xyz="0 0 0" rpy="0 0 0"/>
     </joint>
     <joint name="left_foot_angle" type="fixed">
@@ -557,4 +565,9 @@
                            k_position="${k_position_value_haa}"
                            k_velocity="${k_velocity_value_haa}" />
+    </joint>
+    <joint name="hip_to_world" type="fixed">
+        <parent link="hip_base"/>
+        <child link="${parent_name}"/>
+        <origin xyz="0 0 ${-(lower_leg_height+upper_leg_height+ankle_plate_height+width/2.0+hover_height)}" rpy="0 0 0"/>
     </joint>
     <joint name="right_hip_aa" type="revolute">
